File: Ampli_0_5W.kicad_sch (KiCad schematic)
At the start: 66 parts, among them J1 RF_In, J2 PTT_In, J3 Aux_PTT_Out, J4 RF_Out, Q1 2N7002, Q2 FDD6685, Q3 2N5109, Q4 AFT05MP075N, T1 4:1, T2 1:1, T3 1:9, U1 LM78M05_TO252

Commit message: pennywhistle compatible mounting holes
Other:
- note added: "AFT05MP075N 50W (47 dBm) out Gain : 20 dB P in 0,5W (27 dBm) 2N5109 gain should be at least 18 dB Pout Red pitaya : 7 to 9 dBm"
- note added: "Pennywhistle mounting holes : 90x70mm"
- note removed: "Todo - Vérifier perçages de fixation - Vérifier contact semelle/pcb/gnd"
Changed lines of the file:
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@@
     (effects (font (size 1.27 1.27)) (justify left bottom))
-  )
-  (text "Todo\n- Vérifier perçages de fixation\n- Vérifier contact semelle/pcb/gnd\n"
-    (at 149.225 32.385 0)
-    (effects (font (size 3 3)) (justify left bottom))
   )
   (text "4\n\n4\n" (at 81.915 100.965 0)
@@
     (effects (font (size 1.27 1.27)) (justify left bottom))
   )
+  (text "AFT05MP075N\n50W (47 dBm) out\nGain : 20 dB\nP in 0,5W (27 dBm)\n\n2N5109 gain should be at least 18 dB\nPout Red pitaya : 7 to 9 dBm\n\n"
+    (at 91.44 145.415 0)
+    (effects (font (size 1.27 1.27)) (justify left bottom))
+  )
+  (text "Pennywhistle mounting holes : 90x70mm" (at 160.02 19.685 0)
+    (effects (font (size 1.27 1.27)) (justify left bottom))
+  )
   (text "2xFB61-4852\n3T 25 Ohms coax\n" (at 156.21 109.22 0)
     (effects (font (size 1.27 1.27)) (justify left bottom))
   )
   (text "N.B. FR4, 0,8mm, Er 4.3, Cu 0.035mm\nstrip 50 Ohms à 1.5mm"
-    (at 241.935 22.86 0)
+    (at 160.02 25.4 0)
     (effects (font (size 1.27 1.27)) (justify left bottom))
   )
@@
   (symbol (lib_id "Mechanical:MountingHole_Pad") (at 48.26 41.275 0) (unit 1)
     (in_bom yes) (on_board yes) (dnp no)
-    (property "Reference" "H2" (at -95.885 25.7615 0)
-      (effects (font (size 1.27 1.27)) (justify left))
-    )
-    (property "Value" "MountingHole_Pad" (at -95.885 28.5366 0)
+    (property "Reference" "H2" (at 38.735 41.91 0)
+      (effects (font (size 1.27 1.27)) (justify left))
+    )
+    (property "Value" "MountingHole_Pad" (at 34.925 44.45 0)
       (effects (font (size 1.27 1.27)) (justify left))
     )
@@
       (effects (font (size 1.27 1.27)) (justify left))
     )
-    (property "Value" "MountingHole_Pad" (at 14.605 36.1566 0)
-      (effects (font (size 1.27 1.27)) (justify left))
-    )
+    (property "Value" "MountingHole_Pad" (at 149.86 51.435 0)
+      (effects (font (size 1.27 1.27)) (justify left))
+    )

Commit message: new 3D image, minor changes
Parts:
- added C30: 100n, Capacitor_SMD:C_0603_1608Metric_Pad1.08x0.95mm_HandSolder, symbol Device:C_Small
- added Q5: 2SC5551A, Package_TO_SOT_SMD:SOT-89-3, symbol Transistor_BJT:BCX56
- added R16: 10R, Resistor_SMD:R_0603_1608Metric_Pad0.98x0.95mm_HandSolder, symbol Device:R_Small
Connections:
- net GND: now also C30.1, R16.1
- net at C6.1, Q3.2 (B), R5.1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: now also Q5.1 (B)
- new net: C30.2, Q5.3 (E), R16.2
Other:
- note added: "2SC5551 replacement part ? alternate footprint"
Changed lines of the file:
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@@
   (junction (at 114.935 46.99) (diameter 0) (color 0 0 0 0)
   )
+  (junction (at 82.55 137.795) (diameter 0) (color 0 0 0 0)
+  )
   (junction (at 78.105 114.935) (diameter 0) (color 0 0 0 0)
   )
@@
     (stroke (width 0) (type default))
   )
+  (wire (pts (xy 70.485 107.95) (xy 70.485 109.855))
+    (stroke (width 0) (type default))
+  )
   (wire (pts (xy 142.875 138.43) (xy 146.05 138.43))
     (stroke (width 0) (type default))
@@
     (stroke (width 0) (type default))
   )
+  (wire (pts (xy 70.485 132.715) (xy 74.93 132.715))
+    (stroke (width 0) (type default))
+  )
   (wire (pts (xy 142.875 147.32) (xy 146.05 147.32))
     (stroke (width 0) (type default))
@@
     (stroke (width 0) (type default))
   )
+  (wire (pts (xy 82.55 137.795) (xy 83.82 137.795))
+    (stroke (width 0) (type default))
+  )
   (wire (pts (xy 146.05 142.875) (xy 146.05 138.43))
     (stroke (width 0) (type default))
@@
     (stroke (width 0) (type default))
   )
+  (wire (pts (xy 80.645 103.505) (xy 82.55 103.505))
+    (stroke (width 0) (type default))
+  )
   (wire (pts (xy 90.17 52.705) (xy 91.44 52.705))
     (stroke (width 0) (type default))
   )
+  (wire (pts (xy 83.82 142.875) (xy 83.82 144.145))
+    (stroke (width 0) (type default))
+  )
   (wire (pts (xy 27.305 18.415) (xy 27.305 19.05))
     (stroke (width 0) (type default))
@@
     (stroke (width 0) (type default))
   )
+  (wire (pts (xy 82.55 103.505) (xy 82.55 127.635))
+    (stroke (width 0) (type default))
+  )
   (wire (pts (xy 158.75 51.435) (xy 158.75 52.705))
     (stroke (width 0) (type default))
@@
     (stroke (width 0) (type default))
   )
+  (wire (pts (xy 80.645 137.795) (xy 82.55 137.795))
+    (stroke (width 0) (type default))
+  )
   (wire (pts (xy 73.025 46.99) (xy 114.935 46.99))
     (stroke (width 0) (type default))
@@
     (stroke (width 0) (type default))
   )
+  (wire (pts (xy 70.485 109.855) (xy 70.485 132.715))
+    (stroke (width 0) (type default))
+  )
   (wire (pts (xy 153.035 86.995) (xy 153.035 93.98))
     (stroke (width 0) (type default))
@@
     (stroke (width 0) (type default))
   )
+  (wire (pts (xy 80.645 142.875) (xy 80.645 144.145))
+    (stroke (width 0) (type default))
+  )
   (wire (pts (xy 173.355 93.98) (xy 174.625 93.98))
     (stroke (width 0) (type default))
@@
     (stroke (width 0) (type default))
   )
-  (wire (pts (xy 70.485 107.95) (xy 70.485 109.855))
-    (stroke (width 0) (type default))
-  )
   (wire (pts (xy 90.17 65.405) (xy 90.17 70.485))
     (stroke (width 0) (type default))
@@
     (effects (font (size 1.27 1.27)) (justify left bottom))
   )
+  (text "2SC5551 replacement part ? alternate footprint\n" (at 40.005 142.875 0)
+    (effects (font (size 1.27 1.27)) (justify left bottom))
+  )
   (text "N.B. FR4, 0,8mm, Er 4.3, Cu 0.035mm\nstrip 50 Ohms à 1.5mm"
     (at 160.02 25.4 0)
@@
     )
   )
+  (symbol (lib_id "Device:C_Small") (at 80.645 140.335 180) (unit 1)
+    (in_bom yes) (on_board yes) (dnp no)
+    (property "Reference" "C30" (at 74.295 139.065 0)
+      (effects (font (size 1.27 1.27)) (justify right))
+    )
+    (property "Value" "100n" (at 75.565 142.24 0)
+      (effects (font (size 1.27 1.27)) (justify right))
+    )
+    (property "Footprint" "Capacitor_SMD:C_0603_1608Metric_Pad1.08x0.95mm_HandSolder" (at 80.645 140.335 0)
+      (effects (font (size 1.27 1.27)) hide)
+    )
+    (property "Datasheet" "~" (at 80.645 140.335 0)
+      (effects (font (size 1.27 1.27)) hide)
+    )
+    (pin "1")
+    (pin "2")
+    (instances
+      (project "Ampli_0_5W"
+        (path "/e63e39d7-6ac0-4ffd-8aa3-1841a4541b55"
+          (reference "C30") (unit 1)
+        )
+      )
+    )
+  )
   (symbol (lib_id "power:GND") (at 19.05 19.685 0) (unit 1)
     (in_bom yes) (on_board yes) (dnp no) (fields_autoplaced)
@@
     )
   )
+  (symbol (lib_id "Device:R_Small") (at 83.82 140.335 180) (unit 1)
+    (in_bom yes) (on_board yes) (dnp no)
+    (property "Reference" "R16" (at 85.09 139.7 0)
+      (effects (font (size 1.27 1.27)) (justify right))
+    )
+    (property "Value" "10R" (at 84.455 142.875 0)
+      (effects (font (size 1.27 1.27)) (justify right))
+    )
+    (property "Footprint" "Resistor_SMD:R_0603_1608Metric_Pad0.98x0.95mm_HandSolder" (at 83.82 140.335 0)
+      (effects (font (size 1.27 1.27)) hide)
+    )
+    (property "Datasheet" "~" (at 83.82 140.335 0)
+      (effects (font (size 1.27 1.27)) hide)
+    )
+    (pin "1")
+    (pin "2")
+    (instances
+      (project "Ampli_0_5W"
+        (path "/e63e39d7-6ac0-4ffd-8aa3-1841a4541b55"
+          (reference "R16") (unit 1)
+        )
+      )
+    )
+  )
   (symbol (lib_id "Device:C_Small") (at 151.13 142.875 270) (unit 1)
     (in_bom yes) (on_board yes) (dnp no) (fields_autoplaced)
@@
     )
   )
+  (symbol (lib_id "Transistor_BJT:BCX56") (at 80.01 132.715 0) (unit 1)
+    (in_bom yes) (on_board yes) (dnp no) (fields_autoplaced)
+    (property "Reference" "Q5" (at 84.8614 132.0713 0)
+      (effects (font (size 1.27 1.27)) (justify left))
+    )
+    (property "Value" "2SC5551A" (at 84.8614 133.9923 0)
+      (effects (font (size 1.27 1.27)) (justify left))
+    )
+    (property "Footprint" "Package_TO_SOT_SMD:SOT-89-3" (at 85.09 134.62 0)
+      (effects (font (size 1.27 1.27) italic) (justify left) hide)
+    )
+    (property "Datasheet" "http://cache.nxp.com/documents/data_sheet/BCP56_BCX56_BC56PA.pdf?pspll=1" (at 80.01 132.715 0)
+      (effects (font (size 1.27 1.27)) (justify left) hide)
+    )
+    (pin "1")
+    (pin "2")
+    (pin "3")
+    (instances
+      (project "Ampli_0_5W"
+        (path "/e63e39d7-6ac0-4ffd-8aa3-1841a4541b55"
+          (reference "Q5") (unit 1)
+        )
+      )
+    )
+  )
+  (symbol (lib_id "power:GND") (at 80.645 144.145 0) (unit 1)
+    (in_bom yes) (on_board yes) (dnp no) (fields_autoplaced)
+    (property "Reference" "#PWR016" (at 80.645 150.495 0)
+      (effects (font (size 1.27 1.27)) hide)
+    )
+    (property "Value" "GND" (at 80.645 148.7075 0)
+      (effects (font (size 1.27 1.27)))
+    )
+    (property "Footprint" "" (at 80.645 144.145 0)
+      (effects (font (size 1.27 1.27)) hide)
+    )
+    (property "Datasheet" "" (at 80.645 144.145 0)
+      (effects (font (size 1.27 1.27)) hide)
+    )
+    (pin "1")
+    (instances
+      (project "Ampli_0_5W"
+        (path "/e63e39d7-6ac0-4ffd-8aa3-1841a4541b55"
+          (reference "#PWR016") (unit 1)
+        )
+      )
+    )
+  )
   (symbol (lib_id "Mechanical:MountingHole_Pad") (at 174.625 36.195 0) (unit 1)
     (in_bom yes) (on_board yes) (dnp no) (fields_autoplaced)
@@
         )
       )
+    )
+  )
+  (symbol (lib_id "power:GND") (at 83.82 144.145 0) (unit 1)
+    (in_bom yes) (on_board yes) (dnp no) (fields_autoplaced)
+    (property "Reference" "#PWR041" (at 83.82 150.495 0)
+      (effects (font (size 1.27 1.27)) hide)
+    )
+    (property "Value" "GND" (at 83.82 148.7075 0)
+      (effects (font (size 1.27 1.27)))
+    )
+    (property "Footprint" "" (at 83.82 144.145 0)
+      (effects (font (size 1.27 1.27)) hide)
+    )
+    (property "Datasheet" "" (at 83.82 144.145 0)
+      (effects (font (size 1.27 1.27)) hide)
+    )
+    (pin "1")
+    (instances
+      (project "Ampli_0_5W"
+        (path "/e63e39d7-6ac0-4ffd-8aa3-1841a4541b55"
+          (reference "#PWR041") (unit 1)
+        )
+      )
